Commit message: Solve bug somthing

File: zeabus_model/urdf/zeabus_robot.urdf (robot description, URDF)
Before this commit: robot zeabus_robot, 1 links, 0 joints
Links:
- removed link base_link_robot
- added link base_link; visual cylinder length=0.15 radius=0.12; visual cylinder length=0.92 radius=0.105
- added link bottom_camera
- added link bottom_camera_optical_frame
Joints:
- added joint base_link_bottom_camera: type fixed, parent base_link, child bottom_camera, origin xyz=0.26 0 0 rpy=0 ${PI / 2 } 0
- added joint bottom_camera_to_optical_frame: type fixed, parent bottom_camera, child bottom_camera_optical_frame, origin xyz=0 0 0 rpy=${-1.0 * PI / 2} 0 ${-1.0 * PI / 2}
