Commit message: OK Path

File: zeabus_model/urdf/path.urdf (robot description, URDF)
Before this commit: robot mission_path, 2 links, 1 joints
Joints:
- joint base_path_to_path: origin xyz=-0.62 -0.5 0.0 rpy=${-1 * PI / 2 } 0 0 -> xyz=0 -0.5 0.0 rpy=${-1 * PI / 2 } 0 0

Commit message: Waiting to test

File: zeabus_model/urdf/path.urdf (robot description, URDF)
Before this commit: robot mission_path, 2 links, 1 joints
Joints:
- joint base_path_to_path: origin xyz=0 -0.5 0.0 rpy=${-1 * PI / 2 } 0 0 -> xyz=0.5 0.0 0.0 rpy=${-1 * PI / 2 } 0 ${ PI / 2 }
