Commit message: Add frame wait stl file

File: zeabus_model/urdf/zeabus.urdf (robot description, URDF)
Before this commit: robot mission_path, 4 links, 3 joints
Links:
- added link front_camera
- added link front_camera_optical_frame
Joints:
- added joint base_link_front_camera: type fixed, parent base_link, child front_camera, origin xyz=0.43 0 0 rpy=0 0 0
- added joint front_camera_to_optical_frame: type fixed, parent front_camera, child front_camera_optical_frame, origin xyz=0 0 0 rpy=${-1.0 * PI / 2} 0 ${-1.0 * PI / 2}
- joint base_link_bottom_camera: parent link -> base_link

Commit message: Edit coordinate frame

File: zeabus_model/urdf/zeabus.urdf (robot description, URDF)
Before this commit: robot mission_path, 6 links, 5 joints
Links:
- removed link bottom_camera_optical_frame
- removed link front_camera_optical_frame
- added link bottom_camera_optical
- added link front_camera_optical
Joints:
- joint bottom_camera_to_optical_frame: child bottom_camera_optical_frame -> bottom_camera_optical; origin xyz=0 0 0 rpy=${-1.0 * PI / 2} 0 ${-1.0 * PI / 2} -> xyz=0 0 0 rpy=0 ${-1.0 * PI / 2} ${-1.0 * PI / 2}
- joint front_camera_to_optical_frame: child front_camera_optical_frame -> front_camera_optical; origin xyz=0 0 0 rpy=${-1.0 * PI / 2} 0 ${-1.0 * PI / 2} -> xyz=0 0 0 rpy=0 ${PI / 2} ${-1.0 * PI / 2}

Commit message: Finish fix all camera frame

File: zeabus_model/urdf/zeabus.urdf (robot description, URDF)
Before this commit: robot mission_path, 6 links, 5 joints
Joints:
- joint bottom_camera_to_optical_frame: origin xyz=0 0 0 rpy=0 ${-1.0 * PI / 2} ${-1.0 * PI / 2} -> xyz=0 0 0 rpy=${PI / 2} 0 ${ PI / -2}
- joint front_camera_to_optical_frame: origin xyz=0 0 0 rpy=0 ${PI / 2} ${-1.0 * PI / 2} -> xyz=0 0 0 rpy=${PI / 2} 0 ${ PI / -2}
