Commit message: Edit urdf one mode one link

File: zeabus_model/urdf/flag.urdf (robot description, URDF)
Before this commit: robot flag, 2 links, 1 joints
Links:
- removed link flage_target_header
- link flag_target: geometry visual box size=0.4 0.1 0.08; visual cylinder length=0.65 radius=0.05
Joints:
- removed joint flag_connect

File: zeabus_model/urdf/zeabus_robot.urdf (robot description, URDF)
Before this commit: robot zeabus_robot, 2 links, 1 joints
Links:
- removed link base_link_header
- link base_link_robot: geometry visual cylinder length=0.15 radius=0.12; visual cylinder length=0.92 radius=0.105
Joints:
- removed joint point_header_robot

Commit message: Edit about model

File: zeabus_model/urdf/flag.urdf (robot description, URDF)
Before this commit: robot flag, 1 links, 0 joints
Links:
- removed link flag_target
- added link base_link_target; visual box size=0.4 0.1 0.08; visual cylinder length=0.65 radius=0.05

Commit message: Update after test

File: zeabus_model/urdf/flag.urdf (robot description, URDF)
Before this commit: robot flag, 2 links, 1 joints
Links:
- removed link flag_target
- removed link flage_target_header
- added link base_link_target; visual box size=0.4 0.1 0.08; visual cylinder length=0.65 radius=0.05
Joints:
- removed joint flag_connect
